Commit message: Fix STL mesh paths and define end-effector frame in URDF

File: description/urdf/open_manipulator_y.urdf (robot description, URDF)
Before this commit: robot open_manipulator_y, 14 links, 13 joints
Links:
- added link tcp_link; visual sphere radius=0.005
- link end_effector_flange_link: geometry collision mesh filename=meshs/om_y/flange.stl scale=0.001 0.001 0.001; visual mesh filename=meshs/om_y/flange.stl scale=0.001 0.001 0.001
- link link0: geometry collision mesh filename=meshs/om_y/base_unit.stl scale=0.001 0.001 0.001; visual mesh filename=meshs/om_y/base_unit.stl scale=0.001 0.001 0.001
- link link1: geometry collision mesh filename=meshs/om_y/link1.stl scale=0.001 0.001 0.001; visual mesh filename=meshs/om_y/link1.stl scale=0.001 0.001 0.001
- link link2: geometry collision mesh filename=meshs/om_y/link2.stl scale=0.001 0.001 0.001; visual mesh filename=meshs/om_y/link2.stl scale=0.001 0.001 0.001
- link link3: geometry collision mesh filename=meshs/om_y/link3.stl scale=0.001 0.001 0.001; visual mesh filename=meshs/om_y/link3.stl scale=0.001 0.001 0.001
- link link4: geometry collision mesh filename=meshs/om_y/link4.stl scale=0.001 0.001 0.001; visual mesh filename=meshs/om_y/link4.stl scale=0.001 0.001 0.001
- link link5: geometry collision mesh filename=meshs/om_y/link5.stl scale=0.001 0.001 0.001; visual mesh filename=meshs/om_y/link5.stl scale=0.001 0.001 0.001
- link rh_p12_rn_base: geometry collision mesh filename=meshs/rh_p12_rn_a/base.stl scale=0.001 0.001 0.001; visual mesh filename=meshs/rh_p12_rn_a/base.stl scale=0.001 0.001 0.001
- link rh_p12_rn_l1: geometry collision mesh filename=meshs/rh_p12_rn_a/l1.stl scale=0.001 0.001 0.001; visual mesh filename=meshs/rh_p12_rn_a/l1.stl scale=0.001 0.001 0.001
- link rh_p12_rn_l2: geometry collision mesh filename=meshs/rh_p12_rn_a/l2.stl scale=0.001 0.001 0.001; visual mesh filename=meshs/rh_p12_rn_a/l2.stl scale=0.001 0.001 0.001
- link rh_p12_rn_r1: geometry collision mesh filename=meshs/rh_p12_rn_a/r1.stl scale=0.001 0.001 0.001; visual mesh filename=meshs/rh_p12_rn_a/r1.stl scale=0.001 0.001 0.001
- link rh_p12_rn_r2: geometry collision mesh filename=meshs/rh_p12_rn_a/r2.stl scale=0.001 0.001 0.001; visual mesh filename=meshs/rh_p12_rn_a/r2.stl scale=0.001 0.001 0.001
Joints:
- added joint tcp_joint: type fixed, parent link6, child tcp_link, origin xyz=0 0 0 rpy=0 0 0
